File: LED_Board.sch (KiCad schematic (older format))
At the start: 19 parts, among them J1 Conn_01x06, J2 Conn_01x02, SW1 SW_Push, U1 PCA9531PW_LED_Driver_i2c

Commit message: Added schematic, PCB, etc
As manufactured (v1)
Parts:
- added R10, R11, R12, R13, R14, R15: 100k, Resistors_SMD:R_1206_HandSoldering, symbol R
- added R16: 10k, Resistors_SMD:R_1206_HandSoldering, symbol R
- R1, R2, R8: value R -> 10k
Connections:
- net GND: no longer U1.1 (A0)
- net SCL: now also R1.2, U1.14 (SCL)
- net SDA: now also R2.2, U1.15 (SDA)
- net VDD: now also R10.1, R11.1, R12.1, R13.1, R14.1, R15.1, R16.1
- net ~RESET: now also R16.2
- net at D6.1 (K), U1.10 (LED5): now also R15.2
- net at D1.1 (K), U1.4 (LED0): now also R10.2
- net at D2.1 (K), U1.5 (LED1): now also R11.2
- net at D3.1 (K), U1.6 (LED2): now also R12.2
- net at D4.1 (K), U1.7 (LED3): now also R13.2
- net at D5.1 (K), U1.9 (LED4): now also R14.2
- net A0: now reaches J1.5 (Pin_5)
- net A0: now also U1.1 (A0)
Other:
- moved on the sheet: D2, D3, D4, D5, D6, R4, R5, R6, R7, R9
